Commit message: Remove dependencies

File: gym/envs/gazebo/assets/urdf/kobuki_urdf/urdf/sensors/lidar_sensor.urdf.xacro (robot description, xacro)
@@ -17,7 +17,4 @@
         <geometry>
           <!--<box size="0.01 0.01 0.01" /> -->
-          <!-- <mesh filename="package://rotors_description/meshes/sonar_sensor/max_sonar_ez4.dae"/> -->
-           <!--<mesh filename="package://ardupilot_sitl_gazebo_plugin/meshes/${sensor_mesh}"/>-->
-         <!-- <mesh filename="package://ardupilot_sitl_gazebo_plugin/meshes/lidar_lite_v2/meshes/lidar_lite_v2.dae"/> -->
         </geometry>
       </visual>
@@ -56,13 +53,8 @@
           </range>
         </ray>
-        <plugin name="gazebo_ros_${name}_controller" filename="librotors_gazebo_sonar_plugin.so">
-          <gaussianNoise>0.005</gaussianNoise>
-          <topicName>${ros_topic}</topicName>
-          <frameId>${name}_link</frameId>
-        </plugin>
-	<plugin name="gazebo_ros_${name}_controller" filename="libgazebo_ros_laser.so">
+  <plugin name="gazebo_ros_${name}_controller" filename="libgazebo_ros_laser.so">
           <topicName>/scan</topicName>
           <frameName>${name}_link</frameName>
-	</plugin>
+  </plugin>
       </sensor>
     </gazebo>

Commit message: fix geometry error at launch

File: gym/envs/gazebo/assets/urdf/kobuki_urdf/urdf/sensors/lidar_sensor.urdf.xacro (robot description, xacro)
@@ -15,7 +15,7 @@
       <visual>
         <origin xyz="0 0 0" rpy="0 0 0" />
-        <geometry>
+        <!--<geometry>-->
           <!--<box size="0.01 0.01 0.01" /> -->
-        </geometry>
+        <!--</geometry>-->
       </visual>
    <!--   <collision>

Commit message: launch error fix

File: gym/envs/gazebo/assets/urdf/kobuki_urdf/urdf/sensors/lidar_sensor.urdf.xacro (robot description, xacro)
@@ -13,10 +13,13 @@
         <inertia ixx="0.000000017" ixy="0" ixz="0" iyy="0.000000017" iyz="0" izz="0.000000017" />
       </inertial>
-      <visual>
-        <origin xyz="0 0 0" rpy="0 0 0" />
+      <!--<visual>-->
+        <!--<origin xyz="0 0 0" rpy="0 0 0" />-->
         <!--<geometry>-->
           <!--<box size="0.01 0.01 0.01" /> -->
+          <!-- <mesh filename="package://rotors_description/meshes/sonar_sensor/max_sonar_ez4.dae"/> -->
+           <!--<mesh filename="package://ardupilot_sitl_gazebo_plugin/meshes/${sensor_mesh}"/>-->
+         <!-- <mesh filename="package://ardupilot_sitl_gazebo_plugin/meshes/lidar_lite_v2/meshes/lidar_lite_v2.dae"/> -->
         <!--</geometry>-->
-      </visual>
+      <!--</visual>-->
    <!--   <collision>
         <origin xyz="0 0 0" rpy="0 0 0" />
@@ -53,4 +56,9 @@
           </range>
         </ray>
+        <plugin name="gazebo_ros_${name}_controller" filename="librotors_gazebo_sonar_plugin.so">
+          <gaussianNoise>0.005</gaussianNoise>
+          <topicName>${ros_topic}</topicName>
+          <frameId>${name}_link</frameId>
+        </plugin>
   <plugin name="gazebo_ros_${name}_controller" filename="libgazebo_ros_laser.so">
           <topicName>/scan</topicName>

Commit message: Remove commented dependencies

File: gym/envs/gazebo/assets/urdf/kobuki_urdf/urdf/sensors/lidar_sensor.urdf.xacro (robot description, xacro)
@@ -17,7 +17,4 @@
         <!--<geometry>-->
           <!--<box size="0.01 0.01 0.01" /> -->
-          <!-- <mesh filename="package://rotors_description/meshes/sonar_sensor/max_sonar_ez4.dae"/> -->
-           <!--<mesh filename="package://ardupilot_sitl_gazebo_plugin/meshes/${sensor_mesh}"/>-->
-         <!-- <mesh filename="package://ardupilot_sitl_gazebo_plugin/meshes/lidar_lite_v2/meshes/lidar_lite_v2.dae"/> -->
         <!--</geometry>-->
       <!--</visual>-->
