Commit message: small changes in structure

File: gym_gazebo/envs/assets/urdf/new_articulated/new_arm.urdf (robot description, URDF)
Before this commit: robot hans_arm_3joints, 7 links, 6 joints
Links:
- removed link hans_arm_base_link
- added link new_arm_base_link, mass 7.033; collision mesh filename=package://new_arm_description/meshes/H-ROS_Robot_BASE.stl scale=0.001 0.001 0.001; visual mesh filename=package://new_arm_description/meshes/H-ROS_Robot_BASE.stl scale=0.001 0.001 0.001
- link link1: geometry collision mesh filename=package://new_arm_description/meshes/H-ROS_Robot_LINK1.stl scale=0.001 0.001 0.001; visual mesh filename=package://new_arm_description/meshes/H-ROS_Robot_LINK1.stl scale=0.001 0.001 0.001
- link motor1_link: geometry collision mesh filename=package://new_arm_description/meshes/H-ROS_Robot_new1.stl scale=0.001 0.001 0.001; visual mesh filename=package://new_arm_description/meshes/H-ROS_Robot_new1.stl scale=0.001 0.001 0.001
- link motor3_link: geometry collision mesh filename=package://new_arm_description/meshes/H-ROS_Robot_new2.stl scale=0.001 0.001 0.001; visual mesh filename=package://new_arm_description/meshes/H-ROS_Robot_new2.stl scale=0.001 0.001 0.001
- link motor4_link: geometry collision mesh filename=package://new_arm_description/meshes/H-ROS_Robot_LINK2.stl scale=0.001 0.001 0.001; visual mesh filename=package://new_arm_description/meshes/H-ROS_Robot_LINK2.stl scale=0.001 0.001 0.001
- link motor5_link: geometry collision mesh filename=package://new_arm_description/meshes/H-ROS_Robot_new3.stl scale=0.001 0.001 0.001; visual mesh filename=package://new_arm_description/meshes/H-ROS_Robot_new3.stl scale=0.001 0.001 0.001
Joints:
- joint motor1: parent hans_arm_base_link -> new_arm_base_link
- joint world_to_base_joint: child hans_arm_base_link -> new_arm_base_link

File: gym_gazebo/envs/assets/urdf/new_articulated/new_arm.xacro (robot description, xacro)
@@ -4,5 +4,5 @@
 <!-- |    EDITING THIS FILE BY HAND IS NOT RECOMMENDED                                 | -->
 <!-- =================================================================================== -->
-<robot name="hans_arm_3joints" xmlns:xacro="http://ros.org/wiki/xacro">
+<robot name="new_arm_3joints" xmlns:xacro="http://ros.org/wiki/xacro">
   <link name="world">
     <visual>
@@ -15,5 +15,5 @@
     </visual>
   </link>
-  <link name="hans_arm_base_link">
+  <link name="new_arm_base_link">
     <inertial>
       <origin rpy="0 0 0" xyz="8.625E-08 -4.6583E-06 0.03145"/>
@@ -24,18 +24,18 @@
       <origin rpy="0 0 0" xyz="0 0 0"/>
       <geometry>
-        <mesh filename="package://hans_arm_description/meshes/H-ROS_Robot_BASE.stl" scale="0.001 0.001 0.001"/>
-      </geometry>
-      <material name="Gazebo/Grey">
-        <color rgba="0. 0. 0. 1"/>
-      </material>
-    </visual>
-    <collision>
-      <origin rpy="0 0 0" xyz="0 0 0"/>
-      <geometry>
-        <mesh filename="package://hans_arm_description/meshes/H-ROS_Robot_BASE.stl" scale="0.001 0.001 0.001"/>
-      </geometry>
-    </collision>
-  </link>
-  <gazebo reference="hans_arm_base_link">
+        <mesh filename="package://new_arm_description/meshes/H-ROS_Robot_BASE.stl" scale="0.001 0.001 0.001"/>
+      </geometry>
+      <material name="Gazebo/Grey">
+        <color rgba="0. 0. 0. 1"/>
+      </material>
+    </visual>
+    <collision>
+      <origin rpy="0 0 0" xyz="0 0 0"/>
+      <geometry>
+        <mesh filename="package://new_arm_description/meshes/H-ROS_Robot_BASE.stl" scale="0.001 0.001 0.001"/>
+      </geometry>
+    </collision>
+  </link>
+  <gazebo reference="new_arm_base_link">
     <material>Gazebo/Grey</material>
     <selfCollide>False</selfCollide>
@@ -50,14 +50,14 @@
       <origin rpy="0 0 0" xyz="0 0 0"/>
       <geometry>
-        <mesh filename="package://hans_arm_description/meshes/H-ROS_Robot_HANS1.stl" scale="0.001 0.001 0.001"/>
-      </geometry>
-      <material name="Gazebo/Grey">
-        <color rgba="0. 0. 0. 1"/>
-      </material>
-    </visual>
-    <collision>
-      <origin rpy="0 0 0" xyz="0 0 0"/>
-      <geometry>
-        <mesh filename="package://hans_arm_description/meshes/H-ROS_Robot_HANS1.stl" scale="0.001 0.001 0.001"/>
+        <mesh filename="package://new_arm_description/meshes/H-ROS_Robot_new1.stl" scale="0.001 0.001 0.001"/>
+      </geometry>
+      <material name="Gazebo/Grey">
+        <color rgba="0. 0. 0. 1"/>
+      </material>
+    </visual>
+    <collision>
+      <origin rpy="0 0 0" xyz="0 0 0"/>
+      <geometry>
+        <mesh filename="package://new_arm_description/meshes/H-ROS_Robot_new1.stl" scale="0.001 0.001 0.001"/>
       </geometry>
     </collision>
@@ -76,14 +76,14 @@
       <origin rpy="0 0 0" xyz="0 0 0"/>
       <geometry>
-        <mesh filename="package://hans_arm_description/meshes/H-ROS_Robot_LINK1.stl" scale="0.001 0.001 0.001"/>
-      </geometry>
-      <material name="Gazebo/Grey">
-        <color rgba="0. 0. 0. 1"/>
-      </material>
-    </visual>
-    <collision>
-      <origin rpy="0 0 0" xyz="0 0 0"/>
-      <geometry>
-        <mesh filename="package://hans_arm_description/meshes/H-ROS_Robot_LINK1.stl" scale="0.001 0.001 0.001"/>
+        <mesh filename="package://new_arm_description/meshes/H-ROS_Robot_LINK1.stl" scale="0.001 0.001 0.001"/>
+      </geometry>
+      <material name="Gazebo/Grey">
+        <color rgba="0. 0. 0. 1"/>
+      </material>
+    </visual>
+    <collision>
+      <origin rpy="0 0 0" xyz="0 0 0"/>
+      <geometry>
+        <mesh filename="package://new_arm_description/meshes/H-ROS_Robot_LINK1.stl" scale="0.001 0.001 0.001"/>
       </geometry>
     </collision>
@@ -102,14 +102,14 @@
       <origin rpy="0 0 0" xyz="0 0 0"/>
       <geometry>
-        <mesh filename="package://hans_arm_description/meshes/H-ROS_Robot_HANS2.stl" scale="0.001 0.001 0.001"/>
-      </geometry>
-      <material name="Gazebo/Grey">
-        <color rgba="0. 0. 0. 1"/>
-      </material>
-    </visual>
-    <collision>
-      <origin rpy="0 0 0" xyz="0 0 0"/>
-      <geometry>
-        <mesh filename="package://hans_arm_description/meshes/H-ROS_Robot_HANS2.stl" scale="0.001 0.001 0.001"/>
+        <mesh filename="package://new_arm_description/meshes/H-ROS_Robot_new2.stl" scale="0.001 0.001 0.001"/>
+      </geometry>
+      <material name="Gazebo/Grey">
+        <color rgba="0. 0. 0. 1"/>
+      </material>
+    </visual>
+    <collision>
+      <origin rpy="0 0 0" xyz="0 0 0"/>
+      <geometry>
+        <mesh filename="package://new_arm_description/meshes/H-ROS_Robot_new2.stl" scale="0.001 0.001 0.001"/>
       </geometry>
     </collision>
@@ -128,14 +128,14 @@
       <origin rpy="0 0 0" xyz="0 0 0"/>
       <geometry>
-        <mesh filename="package://hans_arm_description/meshes/H-ROS_Robot_LINK2.stl" scale="0.001 0.001 0.001"/>
-      </geometry>
-      <material name="Gazebo/Grey">
-        <color rgba="0. 0. 0. 1"/>
-      </material>
-    </visual>
-    <collision>
-      <origin rpy="0 0 0" xyz="0 0 0"/>
-      <geometry>
-        <mesh filename="package://hans_arm_description/meshes/H-ROS_Robot_LINK2.stl" scale="0.001 0.001 0.001"/>
+        <mesh filename="package://new_arm_description/meshes/H-ROS_Robot_LINK2.stl" scale="0.001 0.001 0.001"/>
+      </geometry>
+      <material name="Gazebo/Grey">
+        <color rgba="0. 0. 0. 1"/>
+      </material>
+    </visual>
+    <collision>
+      <origin rpy="0 0 0" xyz="0 0 0"/>
+      <geometry>
+        <mesh filename="package://new_arm_description/meshes/H-ROS_Robot_LINK2.stl" scale="0.001 0.001 0.001"/>
       </geometry>
     </collision>
@@ -154,14 +154,14 @@
       <origin rpy="0 0 0" xyz="0 0 0"/>
       <geometry>
-        <mesh filename="package://hans_arm_description/meshes/H-ROS_Robot_HANS3.stl" scale="0.001 0.001 0.001"/>
-      </geometry>
-      <material name="Gazebo/Grey">
-        <color rgba="0. 0. 0. 1"/>
-      </material>
-    </visual>
-    <collision>
-      <origin rpy="0 0 0" xyz="0 0 0"/>
-      <geometry>
-        <mesh filename="package://hans_arm_description/meshes/H-ROS_Robot_HANS3.stl" scale="0.001 0.001 0.001"/>
+        <mesh filename="package://new_arm_description/meshes/H-ROS_Robot_new3.stl" scale="0.001 0.001 0.001"/>
+      </geometry>
+      <material name="Gazebo/Grey">
+        <color rgba="0. 0. 0. 1"/>
+      </material>
+    </visual>
+    <collision>
+      <origin rpy="0 0 0" xyz="0 0 0"/>
+      <geometry>
+        <mesh filename="package://new_arm_description/meshes/H-ROS_Robot_new3.stl" scale="0.001 0.001 0.001"/>
       </geometry>
     </collision>
@@ -174,9 +174,9 @@
     <origin rpy="0 0 0" xyz="0 0 0.02"/>
     <parent link="world"/>
-    <child link="hans_arm_base_link"/>
+    <child link="new_arm_base_link"/>
   </joint>
   <joint name="motor1" type="revolute">
     <origin rpy="0 0 0" xyz="0 0 0.00625"/>
-    <parent link="hans_arm_base_link"/>
+    <parent link="new_arm_base_link"/>
     <child link="motor1_link"/>
     <axis xyz="0 0 1"/>
